Commit message: Fix Foxglove viz server, resolve URDF mesh paths, add browser scene

File: test-base/browser_scene.urdf (robot description, URDF)
Before this commit: robot env, 11 links, 10 joints
Links:
- link base_link: geometry collision mesh filename=assets/base_motor_holder_so101_v1.stl; collision mesh filename=assets/base_so101_v2.stl
- link gripper_link: geometry collision mesh filename=assets/sts3215_03a_v1.stl; collision mesh filename=assets/wrist_roll_follower_so101_v1.stl
- link lower_arm_link: geometry collision mesh filename=assets/motor_holder_so101_wrist_v1.stl; collision mesh filename=assets/sts3215_03a_v1.stl
- link moving_jaw_so101_v1_link: geometry collision mesh filename=assets/moving_jaw_so101_v1.stl; visual mesh filename=assets/moving_jaw_so101_v1.stl
- link shoulder_link: geometry collision mesh filename=assets/motor_holder_so101_base_v1.stl; collision mesh filename=assets/rotation_pitch_so101_v1.stl
- link upper_arm_link: geometry collision mesh filename=assets/sts3215_03a_v1.stl; collision mesh filename=assets/upper_arm_so101_v1.stl
- link wrist_link: geometry collision mesh filename=assets/sts3215_03a_no_horn_v1.stl; collision mesh filename=assets/wrist_roll_pitch_so101_v2.stl
