Commit message: Demo 1: Basic Sine wave

File: test-base/final_browser.urdf (robot description, URDF)
Before this commit: robot env, 11 links, 10 joints
Links:
- link base_link: geometry visual mesh filename=http://192.168.0.101:8000/assets/base_motor_holder_so101_v1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; visual mesh filename=http://192.168.0.101:8000/assets/base_so101_v2.stl
- link gripper_link: geometry visual mesh filename=http://192.168.0.101:8000/assets/sts3215_03a_v1.stl; visual mesh filename=http://192.168.0.101:8000/assets/wrist_roll_follower_so101_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
- link lower_arm_link: geometry visual mesh filename=http://192.168.0.101:8000/assets/motor_holder_so101_wrist_v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; visual mesh filename=http://192.168.0.101:8000/assets/sts3215_03a_v1.stl
- link moving_jaw_so101_v1_link: geometry visual mesh filename=http://192.168.0.101:8000/assets/moving_jaw_so101_v1.stl
- link shoulder_link: geometry visual mesh filename=http://192.168.0.101:8000/assets/motor_holder_so101_base_v1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; visual mesh filename=http://192.168.0.101:8000/assets/rotation_pitch_so101_v1.stl
- link upper_arm_link: geometry visual mesh filename=http://192.168.0.101:8000/assets/sts3215_03a_v1.stl; visual mesh filename=http://192.168.0.101:8000/assets/upper_arm_so101_v1.stl
- link wrist_link: geometry visual mesh filename=http://192.168.0.101:8000/assets/sts3215_03a_no_horn_v1.stl; visual mesh filename=http://192.168.0.101:8000/assets/wrist_roll_pitch_so101_v2.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
