Commit message: fix: restore digital twin bridge, add dynamic URDF IP patch
- start_gesture_demo.sh: replace foxglove-bridge snap restart with
  so101_digital_twin.py background process (port 8765). The snap only
  forwards ROS2 topics; the Python script is required for FK transforms
  and FrameTransforms streaming to Foxglove.
- start_gesture_demo.sh: add sed patch that rewrites all 17 mesh URLs
  in final_twin.urdf from hardcoded Rubik Pi IP (192.168.0.101) to the
  current device IP at launch time. Fixes broken URDF in Foxglove.
- start_gesture_demo.sh: add TWIN_PID to cleanup() so digital twin
  process is properly killed on Ctrl+C.
- final_twin.urdf: pre-patched to current Orin IP (192.168.0.181).
  Script will keep this updated dynamically on every run.

File: final_twin.urdf (robot description, URDF)
Before this commit: robot env, 11 links, 10 joints
Links:
- link base_link: geometry visual mesh filename=http://192.168.0.181:8080/assets/base_motor_holder_so101_v1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; visual mesh filename=http://192.168.0.181:8080/assets/base_so101_v2.stl
- link gripper_link: geometry visual mesh filename=http://192.168.0.181:8080/assets/sts3215_03a_v1.stl; visual mesh filename=http://192.168.0.181:8080/assets/wrist_roll_follower_so101_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
- link lower_arm_link: geometry visual mesh filename=http://192.168.0.181:8080/assets/motor_holder_so101_wrist_v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; visual mesh filename=http://192.168.0.181:8080/assets/sts3215_03a_v1.stl
- link moving_jaw_so101_v1_link: geometry visual mesh filename=http://192.168.0.181:8080/assets/moving_jaw_so101_v1.stl
- link shoulder_link: geometry visual mesh filename=http://192.168.0.181:8080/assets/motor_holder_so101_base_v1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; visual mesh filename=http://192.168.0.181:8080/assets/rotation_pitch_so101_v1.stl
- link upper_arm_link: geometry visual mesh filename=http://192.168.0.181:8080/assets/sts3215_03a_v1.stl; visual mesh filename=http://192.168.0.181:8080/assets/upper_arm_so101_v1.stl
- link wrist_link: geometry visual mesh filename=http://192.168.0.181:8080/assets/sts3215_03a_no_horn_v1.stl; visual mesh filename=http://192.168.0.181:8080/assets/wrist_roll_pitch_so101_v2.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
